File: sensors.kicad_sch (KiCad schematic)
At the start: 9 parts, among them U2 APDS-9306-065, U6 ER_OLEDM0.91_1x-I2C, U7 AM2302

Commit message: feat: implement microSD schematic
Parts:
- removed R12: 4.7K, symbol Device:R
- added J4: Conn_01x04, symbol Connector_Generic:Conn_01x04
Connections:
- net +3V3: now also U7.1 (VDD), J4.1 (Pin_1)
- net GND: now also J4.4 (Pin_4)
- net SENS_SCL: now also J4.2 (Pin_2)
- net SENS_SDA: now also J4.3 (Pin_3)
Other:
- note added: "HEADER_EXPANSION"
