File: storage_sdio.kicad_sch (KiCad schematic)
At the start: 8 parts, among them J5 Micro_SD_Card

Commit message: feat: add can1 can2 schematic
Connections:
- net +3.3V renamed +3V3
Other:
- moved on the sheet: R22, R23, R24, R25, R26
