File: basic_io.kicad_sch (KiCad schematic)
At the start: 12 parts

Commit message: feat: implement sensors schematic
Parts:
- added BZ1: Buzzer, symbol Device:Buzzer
- added JP10, JP11, JP8, JP9: Jumper_2_Open, symbol Jumper:Jumper_2_Open
- added Q2: AO3401A, Package_TO_SOT_SMD:SOT-23, symbol Transistor_FET:AO3401A
- added R14, R15, R16: 10K, symbol Device:R
- added R17: 100, symbol Device:R
- added R18: 100K, symbol Device:R
- added SW3, SW4, SW5: SW_Push, symbol Switch:SW_Push
- R10, R11, R12, R13: value R -> 1K
Connections:
- net GND: now also Q2.2 (S), R18.1, SW3.2, SW4.2, SW5.2
- new net: JP11.2 (B), R17.1, R18.2
- new net: Q2.1 (G), R17.2
- new net: JP10.1 (A), R16.2, SW5.1
- new net: JP8.1 (A), R14.2, SW3.1
- new net: JP9.1 (A), R15.2, SW4.1
- new net: BZ1.2 (-), Q2.3 (D)
- new net +3.3V: BZ1.1 (+), R14.1, R15.1, R16.1
- new net BTN1_N: JP8.2 (B)
- new net BTN2_N: JP9.2 (B)
- new net BTN3_N: JP10.2 (B)
- new net BUZZER_PWM: JP11.1 (A)
Other:
- note added: "BUTTON"
- note added: "BUZZER"
- note added: "LED"
- moved on the sheet: D2, D3, D4, D5, JP4, JP5, JP6, JP7, R10, R11, R12, R13

Commit message: feat: implement microSD schematic
Parts:
- renumbered JP9 to JP10, JP10 to JP11, JP11 to JP4, JP4 to JP5, JP5 to JP6, JP6 to JP7, JP7 to JP8, JP8 to JP9, R18 to R10, R17 to R11, R10 to R12, R11 to R13, R12 to R14, R13 to R15, R14 to R16, R15 to R17, R16 to R18
Changed lines of the file:
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@@
 			(font
 				(size 2.54 2.54)
-				(thickness 0.254)
+				(thickness 0.508)
 				(bold yes)
 			)
@@
 		(dnp no)
 		(fields_autoplaced yes)
-		(property "Reference" "R18"
+		(property "Reference" "R10"
 			(at 77.47 149.8599 0)
 			(show_name no)
@@
 			(project "STM32F407VET6_Minimum_System"
 				(path "/47aad607-e186-4e6e-a0c1-2ae1e2a2d3f0"
-					(reference "R18")
+					(reference "R10")
 					(unit 1)
 				)
@@
 		(dnp no)
 		(fields_autoplaced yes)
-		(property "Reference" "JP4"
+		(property "Reference" "JP5"
 			(at 68.58 48.26 0)
 			(show_name no)
@@
 			(project "STM32F407VET6_Minimum_System"
 				(path "/47aad607-e186-4e6e-a0c1-2ae1e2a2d3f0"
-					(reference "JP4")
+					(reference "JP5")
 					(unit 1)
 				)
@@
 		(dnp no)
 		(fields_autoplaced yes)
-		(property "Reference" "R17"
+		(property "Reference" "R11"
 			(at 82.55 137.16 90)
 			(show_name no)
@@
 			(project "STM32F407VET6_Minimum_System"
 				(path "/47aad607-e186-4e6e-a0c1-2ae1e2a2d3f0"
-					(reference "R17")
+					(reference "R11")
 					(unit 1)
 				)
@@
 		(dnp no)
 		(fields_autoplaced yes)
-		(property "Reference" "#PWR046"
+		(property "Reference" "#PWR040"
 			(at 99.06 128.27 0)
 			(hide yes)
@@
 			(project "STM32F407VET6_Minimum_System"
 				(path "/47aad607-e186-4e6e-a0c1-2ae1e2a2d3f0"
-					(reference "#PWR046")
+					(reference "#PWR040")
 					(unit 1)
 				)
@@
 		(dnp no)
 		(fields_autoplaced yes)
-		(property "Reference" "#PWR044"
+		(property "Reference" "#PWR047"
 			(at 218.44 71.12 0)
 			(hide yes)
@@
 			(project "STM32F407VET6_Minimum_System"
 				(path "/47aad607-e186-4e6e-a0c1-2ae1e2a2d3f0"
-					(reference "#PWR044")
+					(reference "#PWR047")
 					(unit 1)
 				)
@@
 		(dnp no)
 		(fields_autoplaced yes)
-		(property "Reference" "JP10"
+		(property "Reference" "JP11"
 			(at 237.49 77.4699 90)
 			(show_name no)
@@
 			(project "STM32F407VET6_Minimum_System"
 				(path "/47aad607-e186-4e6e-a0c1-2ae1e2a2d3f0"
-					(reference "JP10")
+					(reference "JP11")
 					(unit 1)
 				)
@@
 		(dnp no)
 		(fields_autoplaced yes)
-		(property "Reference" "R13"
+		(property "Reference" "R15"
 			(at 87.63 80.01 90)
 			(show_name no)
@@
 			(project "STM32F407VET6_Minimum_System"
 				(path "/47aad607-e186-4e6e-a0c1-2ae1e2a2d3f0"
-					(reference "R13")
+					(reference "R15")
 					(unit 1)
 				)
@@
 		(dnp no)
 		(fields_autoplaced yes)
-		(property "Reference" "JP6"
+		(property "Reference" "JP7"
 			(at 68.58 68.58 0)
 			(show_name no)
@@
 			(project "STM32F407VET6_Minimum_System"
 				(path "/47aad607-e186-4e6e-a0c1-2ae1e2a2d3f0"
-					(reference "JP6")
+					(reference "JP7")
 					(unit 1)
 				)
@@
 		(dnp no)
 		(fields_autoplaced yes)
-		(property "Reference" "R11"
+		(property "Reference" "R13"
 			(at 87.63 58.42 90)
 			(show_name no)
@@
 			(project "STM32F407VET6_Minimum_System"
 				(path "/47aad607-e186-4e6e-a0c1-2ae1e2a2d3f0"
-					(reference "R11")
+					(reference "R13")
 					(unit 1)
 				)
@@
 		(dnp no)
 		(fields_autoplaced yes)
-		(property "Reference" "#PWR040"
+		(property "Reference" "#PWR045"
 			(at 196.85 77.47 0)
 			(hide yes)
@@
 			(project "STM32F407VET6_Minimum_System"
 				(path "/47aad607-e186-4e6e-a0c1-2ae1e2a2d3f0"
-					(reference "#PWR040")
+					(reference "#PWR045")
 					(unit 1)
 				)
@@
 		(dnp no)
 		(fields_autoplaced yes)
-		(property "Reference" "#PWR041"
+		(property "Reference" "#PWR043"
 			(at 157.48 71.12 0)
 			(hide yes)
@@
 			(project "STM32F407VET6_Minimum_System"
 				(path "/47aad607-e186-4e6e-a0c1-2ae1e2a2d3f0"
-					(reference "#PWR041")
+					(reference "#PWR043")
 					(unit 1)
 				)
@@
 		(dnp no)
 		(fields_autoplaced yes)
-		(property "Reference" "R12"
+		(property "Reference" "R14"
 			(at 87.63 68.58 90)
 			(show_name no)
@@
 			(project "STM32F407VET6_Minimum_System"
 				(path "/47aad607-e186-4e6e-a0c1-2ae1e2a2d3f0"
-					(reference "R12")
+					(reference "R14")
 					(unit 1)
 				)
@@
 		(dnp no)
 		(fields_autoplaced yes)
-		(property "Reference" "JP7"
+		(property "Reference" "JP8"
 			(at 68.58 80.01 0)
 			(show_name no)
@@
 			(project "STM32F407VET6_Minimum_System"
 				(path "/47aad607-e186-4e6e-a0c1-2ae1e2a2d3f0"
-					(reference "JP7")
+					(reference "JP8")
 					(unit 1)
 				)
@@
 		(dnp no)
 		(fields_autoplaced yes)
-		(property "Reference" "#PWR048"
+		(property "Reference" "#PWR039"
 			(at 74.93 163.83 0)
 			(hide yes)
@@
 			(project "STM32F407VET6_Minimum_System"
 				(path "/47aad607-e186-4e6e-a0c1-2ae1e2a2d3f0"
-					(reference "#PWR048")
+					(reference "#PWR039")
 					(unit 1)
 				)
@@
 		(dnp no)
 		(fields_autoplaced yes)
-		(property "Reference" "R16"
+		(property "Reference" "R18"
 			(at 229.87 63.5 90)
 			(show_name no)
@@
 			(project "STM32F407VET6_Minimum_System"
 				(path "/47aad607-e186-4e6e-a0c1-2ae1e2a2d3f0"
-					(reference "R16")
+					(reference "R18")
 					(unit 1)
 				)
@@
 		(dnp no)
 		(fields_autoplaced yes)
-		(property "Reference" "R10"
+		(property "Reference" "R12"
 			(at 87.63 48.26 90)
 			(show_name no)
@@
 			(project "STM32F407VET6_Minimum_System"
 				(path "/47aad607-e186-4e6e-a0c1-2ae1e2a2d3f0"
-					(reference "R10")
+					(reference "R12")
 					(unit 1)
 				)
@@
 		(dnp no)
 		(fields_autoplaced yes)
-		(property "Reference" "#PWR042"
+		(property "Reference" "#PWR044"
 			(at 160.02 102.87 0)
 			(hide yes)
@@
 			(project "STM32F407VET6_Minimum_System"
 				(path "/47aad607-e186-4e6e-a0c1-2ae1e2a2d3f0"
-					(reference "#PWR042")
+					(reference "#PWR044")
 					(unit 1)
 				)
@@
 		(dnp no)
 		(fields_autoplaced yes)
-		(property "Reference" "R15"
+		(property "Reference" "R17"
 			(at 171.45 95.25 90)
 			(show_name no)
@@
 			(project "STM32F407VET6_Minimum_System"
 				(path "/47aad607-e186-4e6e-a0c1-2ae1e2a2d3f0"
-					(reference "R15")
+					(reference "R17")
 					(unit 1)
 				)
@@
 		(dnp no)
 		(fields_autoplaced yes)
-		(property "Reference" "R14"
+		(property "Reference" "R16"
 			(at 168.91 63.5 90)
 			(show_name no)
@@
 			(project "STM32F407VET6_Minimum_System"
 				(path "/47aad607-e186-4e6e-a0c1-2ae1e2a2d3f0"
-					(reference "R14")
+					(reference "R16")
 					(unit 1)
 				)
@@
 		(dnp no)
 		(fields_autoplaced yes)
-		(property "Reference" "JP5"
+		(property "Reference" "JP6"
 			(at 68.58 58.42 0)
 			(show_name no)
@@
 			(project "STM32F407VET6_Minimum_System"
 				(path "/47aad607-e186-4e6e-a0c1-2ae1e2a2d3f0"
-					(reference "JP5")
+					(reference "JP6")
 					(unit 1)
 				)
@@
 		(dnp no)
 		(fields_autoplaced yes)
-		(property "Reference" "#PWR013"
+		(property "Reference" "#PWR042"
 			(at 116.84 95.25 0)
 			(hide yes)
@@
 			(project "STM32F407VET6_Minimum_System"
 				(path "/47aad607-e186-4e6e-a0c1-2ae1e2a2d3f0"
-					(reference "#PWR013")
+					(reference "#PWR042")
 					(unit 1)
 				)
@@
 		(dnp no)
 		(fields_autoplaced yes)
-		(property "Reference" "#PWR047"
+		(property "Reference" "#PWR041"
 			(at 99.06 161.29 0)
 			(hide yes)
@@
 			(project "STM32F407VET6_Minimum_System"
 				(path "/47aad607-e186-4e6e-a0c1-2ae1e2a2d3f0"
-					(reference "#PWR047")
+					(reference "#PWR041")
 					(unit 1)
 				)
@@
 		(dnp no)
 		(fields_autoplaced yes)
-		(property "Reference" "#PWR043"
+		(property "Reference" "#PWR046"
 			(at 199.39 109.22 0)
 			(hide yes)
@@
 			(project "STM32F407VET6_Minimum_System"
 				(path "/47aad607-e186-4e6e-a0c1-2ae1e2a2d3f0"
-					(reference "#PWR043")
+					(reference "#PWR046")
 					(unit 1)
 				)
@@
 		(dnp no)
 		(fields_autoplaced yes)
-		(property "Reference" "JP8"
+		(property "Reference" "JP9"
 			(at 176.53 77.4699 90)
 			(show_name no)
@@
 			(project "STM32F407VET6_Minimum_System"
 				(path "/47aad607-e186-4e6e-a0c1-2ae1e2a2d3f0"
-					(reference "JP8")
+					(reference "JP9")
 					(unit 1)
 				)
@@
 		(dnp no)
 		(fields_autoplaced yes)
-		(property "Reference" "#PWR045"
+		(property "Reference" "#PWR048"
 			(at 257.81 77.47 0)
 			(hide yes)
@@
 			(project "STM32F407VET6_Minimum_System"
 				(path "/47aad607-e186-4e6e-a0c1-2ae1e2a2d3f0"
-					(reference "#PWR045")
+					(reference "#PWR048")
 					(unit 1)
 				)
@@
 		(dnp no)
 		(fields_autoplaced yes)
-		(property "Reference" "JP9"
+		(property "Reference" "JP10"
 			(at 179.07 109.2199 90)
 			(show_name no)
@@
 			(project "STM32F407VET6_Minimum_System"
 				(path "/47aad607-e186-4e6e-a0c1-2ae1e2a2d3f0"
-					(reference "JP9")
+					(reference "JP10")
 					(unit 1)
 				)
@@
 		(dnp no)
 		(fields_autoplaced yes)
-		(property "Reference" "JP11"
+		(property "Reference" "JP4"
 			(at 67.31 137.16 0)
 			(show_name no)
@@
 			(project "STM32F407VET6_Minimum_System"
 				(path "/47aad607-e186-4e6e-a0c1-2ae1e2a2d3f0"
-					(reference "JP11")
+					(reference "JP4")
 					(unit 1)
 				)

Commit message: feat: add can1 can2 schematic
Parts:
- removed Q2: AO3401A, Package_TO_SOT_SMD:SOT-23, symbol Transistor_FET:AO3401A
- added Q3: BUK9832-55A, Package_TO_SOT_SMD:SOT-223-3_TabPin2, symbol Transistor_FET:BUK9832-55A
Connections:
- net GND: now also Q3.3 (S)
- net at R11.2: now also Q3.1 (G)
- net at BZ1.2 (-): now also Q3.2 (D)
Changed lines of the file:
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@@
+	)
+	(symbol
+		(lib_id "Transistor_FET:BUK9832-55A")
+		(at 96.52 143.51 0)
+		(unit 1)
+		(body_style 1)
+		(exclude_from_sim no)
+		(in_bom yes)
+		(on_board yes)
+		(in_pos_files yes)
+		(dnp no)
+		(property "Reference" "Q3"
+			(at 102.87 142.2399 0)
+			(show_name no)
+			(do_not_autoplace no)
+			(effects
+				(font
+					(size 1.27 1.27)
+				)
+				(justify left)
+			)
+		)
+		(property "Value" "BUK9832-55A"
+			(at 102.87 144.7799 0)
+			(show_name no)
+			(do_not_autoplace no)
+			(effects
+				(font
+					(size 1.27 1.27)
+				)
+				(justify left)
+			)
+		)
+		(property "Footprint" "Package_TO_SOT_SMD:SOT-223-3_TabPin2"
+			(at 101.6 145.415 0)
+			(hide yes)
+			(show_name no)
+			(do_not_autoplace no)
+			(effects
+				(font
+					(size 1.27 1.27)
+					(italic yes)
+				)
+				(justify left)
+			)
+		)
+		(property "Datasheet" "https://assets.nexperia.com/documents/data-sheet/BUK9832-55A.pdf"
+			(at 101.6 147.32 0)
+			(hide yes)
+			(show_name no)
+			(do_not_autoplace no)
+			(effects
+				(font
+					(size 1.27 1.27)
+				)
+				(justify left)
+			)
+		)
+		(property "Description" "12A Id, 55V Vds, RdsOn 25mOhm, N-Channel Enhancement Mode MOSFET, SOT-223"
+			(at 96.52 143.51 0)
+			(hide yes)
+			(show_name no)
+			(do_not_autoplace no)
+			(effects
+				(font
+					(size 1.27 1.27)
+				)
+			)
+		)
+		(pin "3"
+		)
+		(pin "2"
+		)
+		(pin "1"
+		)
+		(instances
+			(project "STM32F407VET6_Minimum_System"
+				(path "/47aad607-e186-4e6e-a0c1-2ae1e2a2d3f0"
+					(reference "Q3")
+					(unit 1)
+				)
+			)
+		)
 	)
 	(symbol
@@
 					(unit 1)
 				)
-			)
-		)
-	)
-	(symbol
-		(lib_id "Transistor_FET:AO3401A")
-		(at 96.52 143.51 0)
-		(unit 1)
-		(body_style 1)
-		(exclude_from_sim no)
-		(in_bom yes)
-		(on_board yes)
-		(in_pos_files yes)
-		(dnp no)
-		(fields_autoplaced yes)
-		(property "Reference" "Q2"
-			(at 102.87 142.2399 0)
-			(show_name no)
-			(do_not_autoplace no)
-			(effects
-				(font
-					(size 1.27 1.27)
-				)
-				(justify left)
-			)
-		)
-		(property "Value" "AO3401A"
-			(at 102.87 144.7799 0)
-			(show_name no)
-			(do_not_autoplace no)
-			(effects
-				(font
-					(size 1.27 1.27)
-				)
-				(justify left)
-			)
-		)
-		(property "Footprint" "Package_TO_SOT_SMD:SOT-23"
-			(at 101.6 145.415 0)
-			(hide yes)
-			(show_name no)
-			(do_not_autoplace no)
-			(effects
-				(font
-					(size 1.27 1.27)
-					(italic yes)
-				)
-				(justify left)
-			)
-		)
-		(property "Datasheet" "http://www.aosmd.com/pdfs/datasheet/AO3401A.pdf"
-			(at 101.6 147.32 0)
-			(hide yes)
-			(show_name no)
-			(do_not_autoplace no)
-			(effects
-				(font
-					(size 1.27 1.27)
-				)
-				(justify left)
-			)
-		)
-		(property "Description" "-4.0A Id, -30V Vds, P-Channel MOSFET, SOT-23"
-			(at 96.52 143.51 0)
-			(hide yes)
-			(show_name no)
-			(do_not_autoplace no)
-			(effects
-				(font
-					(size 1.27 1.27)
-				)
-			)
-		)
-		(pin "2"
-		)
-		(pin "1"
-		)
-		(pin "3"
-		)
-		(instances
-			(project "STM32F407VET6_Minimum_System"
-				(path "/47aad607-e186-4e6e-a0c1-2ae1e2a2d3f0"
-					(reference "Q2")
-					(unit 1)
-				)

Commit message: feat: implement analog and timer block
Connections:
- net +3.3V renamed +3V3
