File: onboard_debugger.kicad_sch (KiCad schematic)
At the start: 27 parts, among them J1 USB_C_Receptacle_USB2.0_16P, J2 Conn_01x05, SW2 SW_Push, U2 AMS1117-3.3, U3 USBLC6-2SC6, U4 STM32F103C8Tx, Y2 8MHz

Commit message: feat: implement analog and timer block
Connections:
- net +3V3 is gone; now on net +3V3_DBG: J2.1 (Pin_1)
- net TGT_NRST_DRV: now also U4.46 (PB9); no longer U4.43 (PB7)
- net TGT_SWCLK_DRV: now also U4.45 (PB8); no longer U4.46 (PB9)
- net TGT_SWDIO_DRV: now also U4.43 (PB7); no longer U4.45 (PB8)
Changed lines of the file:
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@@
 	)
 	(label "TGT_SWCLK_DRV"
-		(at 143.51 99.06 180)
+		(at 143.51 96.52 180)
 		(effects
 			(font
@@
 	)
 	(label "TGT_SWDIO_DRV"
-		(at 143.51 96.52 180)
+		(at 143.51 93.98 180)
 		(effects
 			(font
@@
 	)
 	(label "TGT_NRST_DRV"
-		(at 143.51 93.98 180)
+		(at 143.51 99.06 180)
 		(effects
 			(font
@@
 			)
 		)
-		(property "Value" "+3V3"
+		(property "Value" "+3V3_DBG"
 			(at 236.22 88.9 0)
 			(show_name no)
