File: analog_timer.kicad_sch (KiCad schematic)
At the start: 18 parts, among them J10 Conn_01x08, J11 Conn_01x04, J12 Conn_01x02, J8 Conn_01x06, J9 Conn_01x04

Commit message: feat: implement precision adc
Parts:
- C40, C41, C42: value C -> 10nF
- R33, R34, R35: value R -> 1K
- R38, R39: value R -> 47
Connections:
- net PWM1: no longer R37.2, R38.2, R39.2
- new net PWM2: R37.2
- new net PWM3: R39.2
- new net PWM4: R38.2
Changed lines of the file:
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@@
 		)
 	)
-	(global_label "PWM1"
+	(global_label "PWM4"
 		(shape input)
 		(at 212.09 53.34 0)
@@
 		)
 	)
-	(global_label "PWM1"
+	(global_label "PWM3"
 		(shape input)
 		(at 212.09 48.26 0)
@@
 		)
 	)
-	(global_label "PWM1"
+	(global_label "PWM2"
 		(shape input)
 		(at 212.09 43.18 0)
@@
 			)
 		)
-		(property "Value" "C"
+		(property "Value" "10nF"
 			(at 55.88 73.6599 0)
 			(show_name no)
@@
 			)
 		)
-		(property "Value" "C"
+		(property "Value" "10nF"
 			(at 110.49 73.6599 0)
 			(show_name no)
@@
 			)
 		)
-		(property "Value" "R"
+		(property "Value" "1K"
 			(at 97.79 60.96 90)
 			(show_name no)
@@
 			)
 		)
-		(property "Value" "R"
+		(property "Value" "1K"
 			(at 43.18 60.96 90)
 			(show_name no)
@@
 			)
 		)
-		(property "Value" "R"
+		(property "Value" "1K"
 			(at 97.79 29.21 90)
 			(show_name no)
@@
 			)
 		)
-		(property "Value" "C"
+		(property "Value" "10nF"
 			(at 110.49 41.9099 0)
 			(show_name no)
@@
 			)
 		)
-		(property "Value" "R"
+		(property "Value" "47"
 			(at 209.042 52.324 90)
 			(show_name no)
@@
 			)
 		)
-		(property "Value" "R"
+		(property "Value" "47"
 			(at 208.788 47.244 90)
 			(show_name no)
