File: power.kicad_sch (KiCad schematic)
At the start: 18 parts, among them J1 Barrel_Jack, Q1 AO3401A, U10 AP63203WU, U8 AP63205WU, U9 TPS2116DRL

Commit message: feat: add the basic io schematic
Parts:
- C33: value 100uF -> 100nF
Connections:
- net +12V_PROT: now also D1.1 (K); no longer D1.2 (A)
- net GND: now also D1.2 (A); no longer D1.1 (K)
Other:
- moved on the sheet: D1
Changed lines of the file:
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@@
+	(wire
+		(pts
+			(xy 168.91 105.41) (xy 168.91 110.49)
+		)
+		(stroke
+			(width 0)
+			(type default)
+		)
+	)
 	(wire
 		(pts
@@
 		)
 	)
-	(label "+5V_SYS"
-		(at 125.73 110.49 0)
-		(effects
-			(font
-				(size 1.27 1.27)
-			)
-			(justify left bottom)
-		)
-	)
 	(label "PR1"
 		(at 64.77 113.03 0)
@@
 	(label "+12V_PROT"
 		(at 158.75 55.88 0)
-		(effects
-			(font
-				(size 1.27 1.27)
-			)
-			(justify left bottom)
-		)
-	)
-	(label "+5V_SYS"
-		(at 162.56 110.49 0)
 		(effects
 			(font
@@
 			)
 			(justify left bottom)
+		)
+	)
+	(global_label "+5V_SYS"
+		(shape input)
+		(at 125.73 110.49 0)
+		(fields_autoplaced yes)
+		(effects
+			(font
+				(size 1.27 1.27)
+			)
+			(justify left)
+		)
+		(property "Intersheetrefs" "${INTERSHEET_REFS}"
+			(at 137.0609 110.49 0)
+			(hide yes)
+			(show_name no)
+			(do_not_autoplace no)
+			(effects
+				(font
+					(size 1.27 1.27)
+				)
+				(justify left)
+			)
+		)
+	)
+	(global_label "+5V_SYS"
+		(shape input)
+		(at 168.91 105.41 180)
+		(fields_autoplaced yes)
+		(effects
+			(font
+				(size 1.27 1.27)
+			)
+			(justify right)
+		)
+		(property "Intersheetrefs" "${INTERSHEET_REFS}"
+			(at 157.5791 105.41 0)
+			(hide yes)
+			(show_name no)
+			(do_not_autoplace no)
+			(effects
+				(font
+					(size 1.27 1.27)
+				)
+				(justify right)
+			)
 		)
 	)
@@
 	(symbol
 		(lib_id "Device:D_Zener")
-		(at 111.76 64.77 90)
+		(at 111.76 64.77 270)
 		(unit 1)
 		(body_style 1)
@@
 					(size 1.27 1.27)
 				)
-				(justify right)
+				(justify left)
 			)
 		)
@@
 					(size 1.27 1.27)
 				)
-				(justify right)
+				(justify left)
 			)
 		)
@@
 			)
 		)
-		(property "Value" "100uF"
+		(property "Value" "100nF"
 			(at 214.63 107.442 90)
 			(show_name no)

Commit message: feat: implement sensors schematic
Connections:
- net +12V_PROT: now also Q1.3 (D); no longer D1.1 (K), Q1.2 (S)
- net GND: no longer D1.2 (A)
- net at F1.2: now also D1.1 (K), Q1.2 (S); no longer Q1.3 (D)
- net at Q1.1 (G), R2.1: now also D1.2 (A)
Other:
- moved on the sheet: D1, Q1

Commit message: feat: implement microSD schematic
Parts:
- removed R2: 100K, symbol Device:R
- added R9: 100K, symbol Device:R
- renumbered C35 to C27, C31 to C28, C32 to C29, C33 to C30, C30 to C31, C34 to C32, J1 to J3, R8 to R7, R9 to R8, U9 to U5, U8 to U6, U10 to U7
Connections:
- net +12V_PROT: now also D1.1 (K), Q1.2 (S); no longer Q1.3 (D)
- net GND: now also D1.2 (A), R9.2
- net at Q1.1 (G): now also R9.1; no longer D1.2 (A)
- new net: F1.2, Q1.3 (D)
Other:
- moved on the sheet: D1, Q1

Commit message: feat: add can1 can2 schematic
Connections:
- net +3V3: no longer R7.1
- net +5V_EXT: now also R7.1
- net GND: no longer D1.2 (A)
- net at Q1.1 (G), R9.1: now also D1.2 (A)
Other:
- moved on the sheet: D1, R9
Changed lines of the file:
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@@
 	)
 	(junction
-		(at 111.76 53.34)
-		(diameter 0)
-		(color 0 0 0 0)
-	)
-	(junction
-		(at 111.76 71.12)
+		(at 109.22 53.34)
 		(diameter 0)
 		(color 0 0 0 0)
@@
 		(color 0 0 0 0)
 	)
+	(junction
+		(at 99.06 63.5)
+		(diameter 0)
+		(color 0 0 0 0)
+	)
 	(no_connect
 		(at 111.76 120.65)
@@
 	(wire
 		(pts
+			(xy 99.06 74.93) (xy 99.06 77.47)
+		)
+		(stroke
+			(width 0)
+			(type default)
+		)
+	)
+	(wire
+		(pts
 			(xy 223.52 60.96) (xy 223.52 49.53)
 		)
@@
 	(wire
 		(pts
-			(xy 111.76 53.34) (xy 111.76 60.96)
-		)
-		(stroke
-			(width 0)
-			(type default)
-		)
-	)
-	(wire
-		(pts
 			(xy 50.8 123.19) (xy 50.8 129.54)
 		)
@@
 	(wire
 		(pts
-			(xy 111.76 71.12) (xy 111.76 68.58)
-		)
-		(stroke
-			(width 0)
-			(type default)
-		)
-	)
-	(wire
-		(pts
 			(xy 214.63 111.76) (xy 218.44 111.76)
 		)
@@
 	(wire
 		(pts
+			(xy 109.22 53.34) (xy 116.84 53.34)
+		)
+		(stroke
+			(width 0)
+			(type default)
+		)
+	)
+	(wire
+		(pts
 			(xy 153.67 67.31) (xy 153.67 71.12)
 		)
@@
 	(wire
 		(pts
+			(xy 99.06 63.5) (xy 99.06 60.96)
+		)
+		(stroke
+			(width 0)
+			(type default)
+		)
+	)
+	(wire
+		(pts
 			(xy 199.39 111.76) (xy 207.01 111.76)
 		)
@@
 	(wire
 		(pts
+			(xy 109.22 53.34) (xy 109.22 55.88)
+		)
+		(stroke
+			(width 0)
+			(type default)
+		)
+	)
+	(wire
+		(pts
 			(xy 194.31 60.96) (xy 223.52 60.96)
 		)
@@
 	(wire
 		(pts
-			(xy 111.76 53.34) (xy 116.84 53.34)
-		)
-		(stroke
-			(width 0)
-			(type default)
-		)
-	)
-	(wire
-		(pts
 			(xy 194.31 55.88) (xy 194.31 49.53)
 		)
@@
 	(wire
 		(pts
-			(xy 99.06 68.58) (xy 99.06 71.12)
-		)
-		(stroke
-			(width 0)
-			(type default)
-		)
-	)
-	(wire
-		(pts
-			(xy 111.76 71.12) (xy 111.76 72.39)
-		)
-		(stroke
-			(width 0)
-			(type default)
-		)
-	)
-	(wire
-		(pts
 			(xy 210.82 58.42) (xy 210.82 49.53)
 		)
@@
 	(wire
 		(pts
-			(xy 104.14 53.34) (xy 111.76 53.34)
+			(xy 104.14 53.34) (xy 109.22 53.34)
 		)
 		(stroke
@@
 	(wire
 		(pts
+			(xy 99.06 63.5) (xy 109.22 63.5)
+		)
+		(stroke
+			(width 0)
+			(type default)
+		)
+	)
+	(wire
+		(pts
 			(xy 184.15 66.04) (xy 184.15 69.85)
 		)
@@
 	(wire
 		(pts
-			(xy 99.06 71.12) (xy 111.76 71.12)
+			(xy 99.06 67.31) (xy 99.06 63.5)
 		)
 		(stroke
@@
 	(label "+3V3"
 		(at 242.57 102.87 0)
+		(effects
+			(font
+				(size 1.27 1.27)
+			)
+			(justify left bottom)
+		)
+	)
+	(label "+5V_EXT"
+		(at 50.8 99.06 0)
 		(effects
 			(font
@@
 	(symbol
 		(lib_id "Device:D_Zener")
-		(at 111.76 64.77 270)
+		(at 109.22 59.69 270)
 		(unit 1)
 		(body_style 1)
@@
 		(fields_autoplaced yes)
 		(property "Reference" "D1"
-			(at 114.3 63.4999 90)
+			(at 111.76 58.4199 90)
 			(show_name no)
 			(do_not_autoplace no)
@@
 		)
 		(property "Value" "8.2V"
-			(at 114.3 66.0399 90)
+			(at 111.76 60.9599 90)
 			(show_name no)
 			(do_not_autoplace no)
@@
 		)
 		(property "Footprint" ""
-			(at 111.76 64.77 0)
+			(at 109.22 59.69 0)
 			(hide yes)
 			(show_name no)
@@
 		)
 		(property "Datasheet" ""
-			(at 111.76 64.77 0)
+			(at 109.22 59.69 0)
 			(hide yes)
 			(show_name no)
@@
 		)
 		(property "Description" "Zener diode"
-			(at 111.76 64.77 0)
+			(at 109.22 59.69 0)
 			(hide yes)
 			(show_name no)
@@
 	)
 	(symbol
-		(lib_id "power:+3V3")
-		(at 50.8 99.06 0)
-		(unit 1)
-		(body_style 1)
-		(exclude_from_sim no)
-		(in_bom yes)
-		(on_board yes)
-		(in_pos_files yes)
-		(dnp no)
-		(fields_autoplaced yes)
-		(property "Reference" "#PWR028"
-			(at 50.8 102.87 0)
-			(hide yes)
-			(show_name no)
-			(do_not_autoplace no)
-			(effects
-				(font
-					(size 1.27 1.27)
-				)
-			)
-		)
-		(property "Value" "+3V3"
-			(at 50.8 93.98 0)
-			(show_name no)
-			(do_not_autoplace no)
-			(effects
-				(font
-					(size 1.27 1.27)
-				)
-			)
-		)
-		(property "Footprint" ""
-			(at 50.8 99.06 0)
-			(hide yes)
-			(show_name no)
-			(do_not_autoplace no)
-			(effects
-				(font
-					(size 1.27 1.27)
-				)
-			)
-		)
-		(property "Datasheet" ""
-			(at 50.8 99.06 0)
-			(hide yes)
-			(show_name no)
-			(do_not_autoplace no)
-			(effects
-				(font
-					(size 1.27 1.27)
-				)
-			)
-		)
-		(property "Description" "Power symbol creates a global label with name \"+3V3\""
-			(at 50.8 99.06 0)
-			(hide yes)
-			(show_name no)
-			(do_not_autoplace no)
-			(effects
-				(font
-					(size 1.27 1.27)
-				)
-			)
-		)
-		(pin "1"
-		)
-		(instances
-			(project "STM32F407VET6_Minimum_System"
-				(path "/a1a27ae1-62b8-4ba2-b58a-69d83d7aab63"
-					(reference "#PWR028")
-					(unit 1)
-				)
-			)
-		)
-	)
-	(symbol
 		(lib_id "Device:C")
 		(at 153.67 63.5 0)
@@
 	(symbol
 		(lib_id "power:GND")
-		(at 111.76 72.39 0)
+		(at 99.06 77.47 0)
 		(unit 1)
 		(body_style 1)
@@
 		(dnp no)
 		(property "Reference" "#PWR032"
-			(at 111.76 78.74 0)
+			(at 99.06 83.82 0)
 			(hide yes)
 			(show_name no)
@@
 		)
 		(property "Value" "GND"
-			(at 116.332 75.184 0)
+			(at 103.632 80.264 0)
 			(show_name no)
 			(do_not_autoplace no)
@@
 		)
 		(property "Footprint" ""
-			(at 111.76 72.39 0)
+			(at 99.06 77.47 0)
 			(hide yes)
 			(show_name no)
@@
 		)
 		(property "Datasheet" ""
-			(at 111.76 72.39 0)
+			(at 99.06 77.47 0)
 			(hide yes)
 			(show_name no)
@@
 		)
 		(property "Description" "Power symbol creates a global label with name \"GND\" , ground"
-			(at 111.76 72.39 0)
+			(at 99.06 77.47 0)
 			(hide yes)
 			(show_name no)
@@
 	(symbol
 		(lib_id "Device:R")
-		(at 99.06 64.77 0)
+		(at 99.06 71.12 0)
 		(unit 1)
 		(body_style 1)
@@
 		(fields_autoplaced yes)
 		(property "Reference" "R9"
-			(at 101.6 63.4999 0)
+			(at 101.6 69.8499 0)
 			(show_name no)
 			(do_not_autoplace no)
@@
 		)
 		(property "Value" "100K"
-			(at 101.6 66.0399 0)
+			(at 101.6 72.3899 0)
 			(show_name no)
 			(do_not_autoplace no)
@@
 		)
 		(property "Footprint" ""
-			(at 97.282 64.77 90)
+			(at 97.282 71.12 90)
 			(hide yes)
 			(show_name no)
@@
 		)
 		(property "Datasheet" ""
-			(at 99.06 64.77 0)
+			(at 99.06 71.12 0)
 			(hide yes)
 			(show_name no)
@@
 		)
 		(property "Description" "Resistor"
-			(at 99.06 64.77 0)
-			(hide yes)
-			(show_name no)
+			(at 99.06 71.12 0)
+			(hide yes)
+			(show_name no)

Commit message: feat: implement analog and timer block
Parts:
- R7: value 15K -> 35K
- R8: value 15K -> 10K
Changed lines of the file:
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@@
 			)
 		)
-		(property "Value" "15K"
+		(property "Value" "10K"
 			(at 53.34 120.6499 0)
 			(show_name no)
@@
 			)
 		)
-		(property "Value" "15K"
+		(property "Value" "35K"
 			(at 53.34 107.9499 0)
 			(show_name no)

Commit message: feat(ethernet): add LAN8720A PHY and RJ45 MagJack schematic
Changed lines of the file:
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@@
+	)
+	(junction
+		(at 248.92 102.87)
+		(diameter 0)
+		(color 0 0 0 0)
 	)
 	(junction
@@
 		(pts
 			(xy 168.91 110.49) (xy 179.07 110.49)
+		)
+		(stroke
+			(width 0)
+			(type default)
+		)
+	)
+	(wire
+		(pts
+			(xy 248.92 97.79) (xy 248.92 102.87)
 		)
 		(stroke
@@
 	(label "+12V"
 		(at 63.5 53.34 0)
-		(effects
-			(font
-				(size 1.27 1.27)
-			)
-			(justify left bottom)
-		)
-	)
-	(label "+3V3"
-		(at 242.57 102.87 0)
 		(effects
 			(font
@@
 					(unit 1)
 				)
+			)
+		)
+	)
+	(symbol
+		(lib_id "power:+3V3")
+		(at 248.92 97.79 0)
+		(unit 1)
+		(body_style 1)
+		(exclude_from_sim no)
+		(in_bom yes)
+		(on_board yes)
+		(in_pos_files yes)
+		(dnp no)
+		(fields_autoplaced yes)
+		(property "Reference" "#PWR0119"
+			(at 248.92 101.6 0)
+			(hide yes)
+			(show_name no)
+			(do_not_autoplace no)
+			(effects
+				(font
+					(size 1.27 1.27)
+				)
+			)
+		)
+		(property "Value" "+3V3"
+			(at 248.92 92.71 0)
+			(show_name no)
+			(do_not_autoplace no)
+			(effects
+				(font
+					(size 1.27 1.27)
+				)
+			)
+		)
+		(property "Footprint" ""
+			(at 248.92 97.79 0)
+			(hide yes)
+			(show_name no)
+			(do_not_autoplace no)
+			(effects
+				(font
+					(size 1.27 1.27)
+				)
+			)
+		)
+		(property "Datasheet" ""
+			(at 248.92 97.79 0)
+			(hide yes)
+			(show_name no)
+			(do_not_autoplace no)
+			(effects
+				(font
+					(size 1.27 1.27)
+				)
+			)
+		)
+		(property "Description" "Power symbol creates a global label with name \"+3V3\""
+			(at 248.92 97.79 0)
+			(hide yes)
+			(show_name no)
+			(do_not_autoplace no)
+			(effects
+				(font
+					(size 1.27 1.27)
+				)
+			)
+		)
+		(pin "1"
+		)
+		(instances
+			(project "STM32F407VET6_Minimum_System"
+				(path "/a1a27ae1-62b8-4ba2-b58a-69d83d7aab63"
+					(reference "#PWR0119")
+					(unit 1)
+				)
